Commit message: feat: chassis contact sensor 추가 및 충돌 감지 인프라 구축
- racecar.xacro: chassis collision 박스 추가, chassis_inertia 별도 링크 제거 후 chassis에 직접 inertial 부여로 fixed-joint lumping 방지
- racecar.gazebo: libgazebo_ros_bumper 기반 contact sensor 추가, disableFixedJointLumping/preserveFixedJoint 설정으로 SDF 변환 시 chassis link 보존
- package.xml: gazebo_msgs 의존성 추가
- lattice_config.yaml: cost weights 중 velocity·time 항목 비활성화(0.0)

File: src/racecar_description/urdf/racecar.xacro (robot description, xacro)
@@ -11,13 +11,24 @@
   <link name="chassis">
     <visual><xacro:chassis_geometry/><material name="${chassis_color}" /></visual>
+    <!-- 차체 외곽 박스: 라이다 광선 평면(z=0.075)보다 낮게 두어 라이다를 막지 않도록 함.
+         크기는 실제 F1tenth 외형(약 0.55 x 0.28 m)에 근사. -->
+    <collision name="chassis_collision">
+      <origin xyz="0.16 0 0.01" rpy="0 0 0"/>
+      <geometry><box size="0.55 0.28 0.05"/></geometry>
+    </collision>
+    <!-- collision 박스 시각화용 (충돌 형상 확인 디버깅) -->
+    <visual name="chassis_collision_visual">
+      <origin xyz="0.16 0 0.01" rpy="0 0 0"/>
+      <geometry><box size="0.55 0.28 0.05"/></geometry>
+      <material name="collision_box_debug">
+        <color rgba="1.0 0.2 0.2 0.35"/>
+      </material>
+    </visual>
+    <!-- chassis에 직접 실제 inertial 부여 → fixed-joint lumping 방지
+         (이전에는 별도 chassis_inertia link에 있었음) -->
+    <inertial><xacro:chassis_inertial_params /></inertial>
   </link>
   <joint name="base_link_joint" type="fixed">
     <origin xyz="0 0 0.05" rpy="0 0 0" /><parent link="base_link" /><child link="chassis" />
-  </joint>
-  <link name="chassis_inertia">
-    <inertial><xacro:chassis_inertial_params /></inertial>
-  </link>
-  <joint name="chassis_inertia_joint" type="fixed">
-    <origin xyz="0 0 0" rpy="0 0 0" /><parent link="chassis" /><child link="chassis_inertia" />
   </joint>
   <!-- 2. 뒷바퀴 설정 (구동축) -->
@@ -80,5 +91,6 @@
   <link name="laser">
     <inertial><xacro:hokuyo_inertial_params /></inertial>
-    <collision><origin xyz="0 0 0"/><geometry><box size="0.1 0.1 0.1"/></geometry></collision>
+    <!-- 라이다 collision은 차량 간 접근을 가로막지 않도록 작게 (4cm 큐브) -->
+    <collision><origin xyz="0 0 0"/><geometry><box size="0.04 0.04 0.04"/></geometry></collision>
     <visual><origin xyz="0 0 0"/><geometry><mesh filename="package://racecar_description/meshes/hokuyo.dae"/></geometry></visual>
   </link>
