Commit message: feat(racecar_description): 차량 후방 라이다 반사판(rear_reflector) URDF 추가 및 Gazebo 재질 연동

File: src/racecar_description/urdf/racecar.xacro (robot description, xacro)
@@ -107,4 +107,26 @@
     <origin xyz="0.39 0 0.04" /><parent link="chassis" /><child link="zed_camera_link" />
   </joint>
+  <!-- 5. 후방 라이다 반사판 (차폭 28cm x 높이 10cm) -->
+  <!-- 자신의 라이다(x=0.265, 135° 한계)에는 닿지 않는 후방 사각(156°)에 위치하며, 뒤차 라이다에는 28cm 전폭으로 확실히 검출됨 -->
+  <link name="rear_reflector">
+    <inertial>
+      <mass value="1e-3" />
+      <inertia ixx="1e-6" ixy="0" ixz="0" iyy="1e-6" iyz="0" izz="1e-6" />
+    </inertial>
+    <visual>
+      <origin xyz="0 0 0" rpy="0 0 0"/>
+      <geometry><box size="0.02 0.28 0.10"/></geometry>
+      <material name="reflector_color"><color rgba="0.1 0.1 0.1 1.0"/></material>
+    </visual>
+    <collision name="rear_reflector_collision">
+      <origin xyz="0 0 0" rpy="0 0 0"/>
+      <geometry><box size="0.02 0.28 0.10"/></geometry>
+    </collision>
+  </link>
+  <joint name="rear_reflector_joint" type="fixed">
+    <origin xyz="-0.05 0 0.075" rpy="0 0 0"/>
+    <parent link="chassis"/>
+    <child link="rear_reflector"/>
+  </joint>
   <!-- 트랜스미션
   <xacro:wheel_transmission name="left_rear_wheel" />
