Commit message: feat: 멀티카 시각화를 위한 차체 색상 파라미터화 및 RViz car2 디스플레이 추가
- racecar.xacro에 color 인자 추가로 차체 색상 동적 설정 지원
- spawn_car.launch.py에 color launch argument 추가 및 xacro 전달
- f1tenth_lattice_gazebo.launch.py에서 car2에 orange 색상 지정
- f1tenth_default.rviz에 car2 LaserScan, RobotModel, 궤적 마커 시각화 추가

Co-Authored-By: Claude Sonnet 4.6 <noreply@anthropic.com>

File: src/racecar_description/urdf/racecar.xacro (robot description, xacro)
@@ -4,9 +4,11 @@
   <xacro:include filename="$(find racecar_description)/urdf/racecar.gazebo" />
   <xacro:arg name="namespace" default="" />
+  <xacro:arg name="color" default="blue" />
+  <xacro:property name="chassis_color" value="$(arg color)" />
   <xacro:racecar_gazebo namespace="$(arg namespace)" />
   <!-- 1. 기본 링크 설정 -->
   <link name="base_link" />
   <link name="chassis">
-    <visual><xacro:chassis_geometry/><material name="blue" /></visual>
+    <visual><xacro:chassis_geometry/><material name="${chassis_color}" /></visual>
   </link>
   <joint name="base_link_joint" type="fixed">

Commit message: feat(sim): 차량 LiDAR 높이 차폭 셸, lattice 상대차 앞부분 +10 cm 마진
- racecar.xacro lidar_body_shell: 차체 박스가 LiDAR 평면보다 낮아 상대차가 4 cm LiDAR 큐브(360 bin 중 2 bin)로만
  보이던 문제 수정. 차폭 0.28 m 셸 → 2.1 m 앞 30빔/10 bin (기하 예상과 일치, 자기 LiDAR 자가-히트 없음)
- lattice_planner: 상대차 충돌 박스를 앞쪽으로만 +0.10 m (차량 모델뿐 아니라 추월 알고리즘 공격성 완화 마진)
- spawn_car / racecar.gazebo: joint_state 폴백을 Gazebo joint_states 와 병합(덮어쓰기 제거), sim time 일치

이 설정으로 재수집한 데이터로 학습한 ego_p08 이 셸 시뮬 10맵에서 충돌없는 추월 69.0 %, 충돌 6.0 % (lattice 55.0/9.5).

Co-Authored-By: Claude Opus 5.5 <noreply@anthropic.com>

File: src/racecar_description/urdf/racecar.xacro (robot description, xacro)
@@ -25,4 +25,19 @@
         <color rgba="1.0 0.2 0.2 0.35"/>
       </material>
+    </visual>
+    <!-- 라이다 높이 차체 셸 (2026-10-20): 위 차체 박스(z 0.035~0.085 world)는 라이다 광선 평면
+         (laser z = chassis+0.075 = 0.125 world)보다 낮아, 상대차가 라이다에는 4 cm 라이다 큐브(2~3 bin)로만
+         보였다(실차는 차폭이 ~20빔으로 보임). 차폭 0.28 m 셸을 광선 평면에 걸치게 두어 상대차가
+         실차처럼 차폭만큼 잡히게 한다. 자기 라이다(x=0.265)가 자기 셸을 보지 않도록 셸은 라이다 뒤쪽
+         x <= 0.115 에만 둔다(±135° 광선이 셸 측면 y=0.14 를 스치는 한계 x=0.125). 풋프린트가 차체 박스
+         안이라 물리 접촉/범퍼 판정은 그대로다. -->
+    <collision name="lidar_body_shell">
+      <origin xyz="0 0 0.075" rpy="0 0 0"/>
+      <geometry><box size="0.23 0.28 0.06"/></geometry>
+    </collision>
+    <visual name="lidar_body_shell_visual">
+      <origin xyz="0 0 0.075" rpy="0 0 0"/>
+      <geometry><box size="0.23 0.28 0.06"/></geometry>
+      <material name="${chassis_color}" />
     </visual>
     <!-- chassis에 직접 실제 inertial 부여 → fixed-joint lumping 방지
